File: Hesu14/Hesu14.kicad_pcb (KiCad board)
At the start: 2 copper layers, 76.2 x 76.2 mm, 34 parts, among them J2 OLED_128x32, U1 RP2040_Zero

Commit message: Update PCB and Case
Parts:
- moved J2 39.5 mm to (111.4, 48.0), turned to 180 degrees
- moved D10 3.47 mm to (110.0, 104.7)
- moved D11 3.47 mm to (129.1, 104.7)
- moved D9 3.47 mm to (91.0, 104.7)
- moved D1 3.47 mm to (91.0, 66.6)
- moved D13 3.47 mm to (129.1, 47.5)
- moved D2 3.47 mm to (110.0, 66.6)
- moved D3 3.47 mm to (129.1, 66.6)
- moved D5 3.47 mm to (91.0, 85.6)
- moved D6 3.47 mm to (110.0, 85.6)
- moved D7 3.47 mm to (129.1, 85.6)
- moved D14 3.39 mm to (148.0, 47.5)
- moved D4 3.31 mm to (148.1, 66.6)
- moved D8 3.12 mm to (148.0, 85.5)
- moved D12 3.11 mm to (148.0, 104.5)
Connections:
- U1 pad 21: VCC -> unconnected-(U1-3V3-Pad21)
- U1 pad 23: unconnected-(U1-5V-Pad23) -> VCC
Routing:
- net SCL: track 9.62 -> 35.1 mm
- net VCC: track 13.0 -> 38.4 mm
- net SDA: track 17.9 -> 41.0 mm
- net GND: track 13.2 -> 34.1 mm
- net Column 1: track 70.5 -> 64.7 mm
- net Row 1: track 70.5 -> 74.7 mm
- net Row 3: track 110.7 -> 114.8 mm
- net Row 2: track 90.6 -> 94.7 mm
- net Net-(D14-A): track 2.38 -> 4.56 mm
- net Net-(D8-A): track 2.44 -> 4.56 mm
- net Net-(D12-A): track 2.44 -> 4.56 mm
- net Net-(D4-A): track 2.44 -> 4.56 mm
- net Row 0: track 57.7 -> 56.4 mm
- net Column 2: track 82.7 -> 83.9 mm
- net Net-(D5-A): track 3.82 -> 4.57 mm
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